File: Stage1.kicad_sch (KiCad schematic)
At the start: 8 parts, among them U201 UA741

Commit message: Sim tests
Parts:
- U201: value UA741 -> OPA827; Spice_Lib_File UA741.301 -> OPA827.LIB; Spice_Model UA741 -> OPA827
Other:
- note added: "2nd order Butterworth Sallen-Key 0.1Hz HPF G=10"
- note removed: "1st Stage 2nd order Butterworth Sallen-Key 0.1Hz HPF G=10"
Changed lines of the file:
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@@
   (junction (at 120.015 81.915) (diameter 0) (color 0 0 0 0)
   )
+  (junction (at 120.015 111.125) (diameter 0) (color 0 0 0 0)
+  )
   (wire (pts (xy 133.35 66.675) (xy 140.335 66.675))
     (stroke (width 0) (type default) (color 0 0 0 0))
@@
     (stroke (width 0) (type default) (color 0 0 0 0))
   )
+  (wire (pts (xy 120.015 111.125) (xy 129.54 111.125))
+    (stroke (width 0) (type default) (color 0 0 0 0))
+  )
   (wire (pts (xy 125.73 66.675) (xy 108.585 66.675))
     (stroke (width 0) (type default) (color 0 0 0 0))
@@
     (stroke (width 0) (type default) (color 0 0 0 0))
   )
-  (wire (pts (xy 120.015 93.98) (xy 120.015 96.52))
+  (wire (pts (xy 120.015 93.98) (xy 120.015 111.125))
+    (stroke (width 0) (type default) (color 0 0 0 0))
+  )
+  (wire (pts (xy 112.395 111.125) (xy 120.015 111.125))
     (stroke (width 0) (type default) (color 0 0 0 0))
   )
@@
     (stroke (width 0) (type default) (color 0 0 0 0))
   )
-  (text "1st Stage\n2nd order Butterworth\nSallen-Key\n0.1Hz HPF\nG=10"
-    (at 90.17 66.04 0)
+  (text "2nd order Butterworth\nSallen-Key\n0.1Hz HPF\nG=10" (at 90.17 66.04 0)
     (effects (font (size 1.27 1.27)) (justify left bottom))
+  )
+  (hierarchical_label "GND" (shape input) (at 112.395 111.125 180)
+    (effects (font (size 1.27 1.27)) (justify right))
   )
   (hierarchical_label "v+" (shape input) (at 137.795 76.835 90)
@@
     (pin "2")
   )
-  (symbol (lib_id "power:GND") (at 120.015 96.52 0) (unit 1)
-    (in_bom yes) (on_board yes) (fields_autoplaced)
-    (property "Reference" "#PWR0201" (id 0) (at 120.015 102.87 0)
-      (effects (font (size 1.27 1.27)) hide)
-    )
-    (property "Value" "GND" (id 1) (at 120.015 101.6 0))
-    (property "Footprint" "" (id 2) (at 120.015 96.52 0)
-      (effects (font (size 1.27 1.27)) hide)
-    )
-    (property "Datasheet" "" (id 3) (at 120.015 96.52 0)
-      (effects (font (size 1.27 1.27)) hide)
-    )
-    (pin "1")
-  )
   (symbol (lib_id "Simulation_SPICE:OPAMP") (at 140.335 84.455 0) (unit 1)
     (in_bom yes) (on_board yes) (fields_autoplaced)
     (property "Reference" "U201" (id 0) (at 149.86 79.756 0))
-    (property "Value" "UA741" (id 1) (at 149.86 82.296 0))
+    (property "Value" "OPA827" (id 1) (at 149.86 82.296 0))
     (property "Footprint" "" (id 2) (at 140.335 84.455 0)
       (effects (font (size 1.27 1.27)) hide)
@@
       (effects (font (size 1.27 1.27)) (justify left) hide)
     )
-    (property "Spice_Model" "UA741" (id 6) (at 140.335 84.455 0)
-      (effects (font (size 1.27 1.27)) hide)
-    )
-    (property "Spice_Lib_File" "UA741.301" (id 7) (at 140.335 84.455 0)
+    (property "Spice_Model" "OPA827" (id 6) (at 140.335 84.455 0)
+      (effects (font (size 1.27 1.27)) hide)
+    )
+    (property "Spice_Lib_File" "OPA827.LIB" (id 7) (at 140.335 84.455 0)
       (effects (font (size 1.27 1.27)) hide)
     )
@@
     (pin "2")
   )
-  (symbol (lib_id "power:GND") (at 129.54 111.125 0) (unit 1)
-    (in_bom yes) (on_board yes) (fields_autoplaced)
-    (property "Reference" "#PWR0202" (id 0) (at 129.54 117.475 0)
-      (effects (font (size 1.27 1.27)) hide)
-    )
-    (property "Value" "~" (id 1) (at 129.54 116.205 0))
-    (property "Footprint" "" (id 2) (at 129.54 111.125 0)
-      (effects (font (size 1.27 1.27)) hide)
-    )
-    (property "Datasheet" "" (id 3) (at 129.54 111.125 0)
-      (effects (font (size 1.27 1.27)) hide)
-    )
-    (pin "1")
-  )
 )
